File: ts15-rpi-shield.kicad_pcb (KiCad board)
At the start: 2 copper layers, 56 x 65 mm, 13 parts, among them CON1 TROPIC01, IC1 TROPIC01_chip, J1 RPI socket

Commit message: project: Add fabrication gerber data and some tuning
Parts:
- added J2: CS select jumper switch, Connector_PinHeader_2.54mm:PinHeader_2x03_P2.54mm_Vertical, F.Cu at (120.5, 96.2)
- moved R3 37.8 mm to (121.8, 105.8)
- moved R2 1.75 mm to (158.5, 113.5)
- renumbered R3 to R2, R2 to R3
Connections:
- J1 pad 22: unconnected-(J1-Pin_22-Pad22) -> /GPIO25
- J1 pad 24: /SPI_CS -> /SPI_CE0
- J1 pad 26: unconnected-(J1-Pin_26-Pad26) -> /SPI_CE1
Routing:
- net /SPI_CE1: track 0.00 -> 74.2 mm
- net /SPI_CE0: track 0.00 -> 67.1 mm
- net /GPIO25: track 0.00 -> 62.1 mm, vias 0 -> 1
- net /SPI_CS: track 58.7 -> 30.8 mm, vias 2 -> 1
- net VCC: track 99.7 -> 105.8 mm
- net +5V: track 0.00 -> 2.54 mm
- net /GPO: track 50.4 -> 52.9 mm
- net /GPIO5: track 5.04 -> 4.31 mm
- net GND: vias 17 -> 37
Other:
- board text added: "CS0"
- board text added: "CS1"
- board text added: "CS2"
